File: kicad_proj/fpga_pre_test.kicad_sch (KiCad schematic)
At the start: 50 parts, among them IC1 ZMR330FTA, IC2 LM3880MFX-1AB_NOPB, IC3 TPS62147RGXT, IC4 TPS62147RGXT, J1 T50201500000G, J2 T50201500000G, Y1 ASDMB-25.000MHZ-XY-T

Commit message: Small fixes on circuit schematic
Parts:
- C1: value 100nF -> 22uF; footprint Capacitor_SMD:C_0603_1608Metric -> Capacitor_SMD:C_1206_3216Metric
- C10, C11: footprint Capacitor_SMD:C_0603_1608Metric -> Capacitor_SMD:C_1206_3216Metric
- C2: footprint Capacitor_SMD:C_1206_3216Metric -> Capacitor_SMD:C_0805_2012Metric
- C4, C6: footprint Capacitor_SMD:C_0603_1608Metric -> Capacitor_SMD:C_0402_1005Metric
- C5, C8: footprint Capacitor_SMD:C_0603_1608Metric -> Capacitor_SMD:C_0805_2012Metric
- C9: footprint Capacitor_SMD:C_0603_1608Metric -> Capacitor_SMD:C_1210_3225Metric
- R12: value 505k -> 205k
- R13: value 135k -> 54.9k
- R16, R17, R18, R19, R20: footprint Resistor_SMD:R_0603_1608Metric -> Resistor_SMD:R_1206_3216Metric
Other:
- note added: "(1.5W Max.)"
- note added: "(3.314V)"
- note removed: "(3.319V)"
- moved on the sheet: R1, R2, S1
Changed lines of the file:
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@@
 	(title_block
 		(title "FPGA Pre Test")
-		(date "2025-10-09")
-		(rev "v1.0.0")
+		(date "2025-10-15")
+		(rev "v1.0.1")
 		(comment 1 "Github: https://github.com/bsiyoung/FPGA_Pre_Test")
 		(comment 2 "Author: Park Siyoung")
@@
 		)
 	)
+	(text "(1.5W Max.)"
+		(exclude_from_sim no)
+		(at 207.264 129.794 0)
+		(effects
+			(font
+				(size 1.27 1.27)
+				(color 0 0 255 1)
+			)
+		)
+	)
 	(text "(2.2uH)"
 		(exclude_from_sim no)
@@
 		)
 	)
-	(text "(3.319V)"
+	(text "(3.314V)"
 		(exclude_from_sim no)
 		(at 127 164.338 0)
@@
 	)
 	(junction
-		(at 181.61 45.72)
+		(at 182.88 48.26)
 		(diameter 0)
 		(color 0 0 0 0)
@@
 	(wire
 		(pts
-			(xy 166.37 48.26) (xy 168.91 48.26)
+			(xy 167.64 50.8) (xy 170.18 50.8)
 		)
 		(stroke
@@
 	(wire
 		(pts
-			(xy 181.61 54.61) (xy 181.61 55.88)
+			(xy 182.88 57.15) (xy 182.88 58.42)
 		)
 		(stroke
@@
 	(wire
 		(pts
-			(xy 168.91 50.8) (xy 166.37 50.8)
+			(xy 170.18 53.34) (xy 167.64 53.34)
 		)
 		(stroke
@@
 	(wire
 		(pts
-			(xy 168.91 55.88) (xy 168.91 50.8)
+			(xy 170.18 58.42) (xy 170.18 53.34)
 		)
 		(stroke
@@
 	(wire
 		(pts
-			(xy 181.61 45.72) (xy 181.61 46.99)
+			(xy 182.88 48.26) (xy 182.88 49.53)
 		)
 		(stroke
@@
 	(wire
 		(pts
-			(xy 166.37 45.72) (xy 181.61 45.72)
+			(xy 167.64 48.26) (xy 182.88 48.26)
 		)
 		(stroke
@@
 	(wire
 		(pts
-			(xy 181.61 44.45) (xy 181.61 45.72)
+			(xy 182.88 46.99) (xy 182.88 48.26)
 		)
 		(stroke
@@
 	(wire
 		(pts
-			(xy 184.15 35.56) (xy 181.61 35.56)
+			(xy 185.42 38.1) (xy 182.88 38.1)
 		)
 		(stroke
@@
 	(wire
 		(pts
-			(xy 181.61 35.56) (xy 181.61 36.83)
+			(xy 182.88 38.1) (xy 182.88 39.37)
 		)
 		(stroke
@@
 	(hierarchical_label "SEQ_EN"
 		(shape output)
-		(at 168.91 48.26 0)
+		(at 170.18 50.8 0)
 		(effects
 			(font
@@
 	(hierarchical_label "3V3LVR"
 		(shape input)
-		(at 184.15 35.56 0)
+		(at 185.42 38.1 0)
 		(effects
 			(font
@@
 	(symbol
 		(lib_id "power:GND")
-		(at 168.91 55.88 0)
+		(at 170.18 58.42 0)
 		(unit 1)
 		(exclude_from_sim no)
@@
 		(dnp no)
 		(property "Reference" "#PWR06"
-			(at 168.91 62.23 0)
+			(at 170.18 64.77 0)
 			(effects
 				(font
@@
 		)
 		(property "Value" "GND"
-			(at 168.91 59.944 0)
+			(at 170.18 62.484 0)
 			(effects
 				(font
@@
 		)
 		(property "Footprint" ""
-			(at 168.91 55.88 0)
+			(at 170.18 58.42 0)
 			(effects
 				(font
@@
 		)
 		(property "Datasheet" ""
-			(at 168.91 55.88 0)
+			(at 170.18 58.42 0)
 			(effects
 				(font
@@
 		)
 		(property "Description" "Power symbol creates a global label with name \"GND\" , ground"
-			(at 168.91 55.88 0)
+			(at 170.18 58.42 0)
 			(effects
 				(font
@@
 	(symbol
 		(lib_id "Device:R")
-		(at 181.61 50.8 0)
+		(at 182.88 53.34 0)
 		(unit 1)
 		(exclude_from_sim no)
@@
 		(dnp no)
 		(property "Reference" "R2"
-			(at 183.134 49.53 0)
+			(at 184.404 52.07 0)
 			(effects
 				(font
@@
 		)
 		(property "Value" "100k"
-			(at 183.134 52.07 0)
+			(at 184.404 54.61 0)
 			(effects
 				(font
@@
 		)
 		(property "Footprint" "Resistor_SMD:R_0603_1608Metric"
-			(at 179.832 50.8 90)
+			(at 181.102 53.34 90)
 			(effects
 				(font
@@
 		)
 		(property "Datasheet" "~"
-			(at 181.61 50.8 0)
+			(at 182.88 53.34 0)
 			(effects
 				(font
@@
 		)
 		(property "Description" "Resistor"
-			(at 181.61 50.8 0)
+			(at 182.88 53.34 0)
 			(effects
 				(font
@@
 			)
 		)
-		(property "Footprint" "Capacitor_SMD:C_0603_1608Metric"
+		(property "Footprint" "Capacitor_SMD:C_0805_2012Metric"
 			(at 106.3752 101.6 0)
 			(effects
@@
 			)
 		)
-		(property "Footprint" "Resistor_SMD:R_0603_1608Metric"
+		(property "Footprint" "Resistor_SMD:R_1206_3216Metric"
 			(at 183.642 134.62 90)
 			(effects
@@
 			)
 		)
-		(property "Footprint" "Capacitor_SMD:C_0603_1608Metric"
+		(property "Footprint" "Capacitor_SMD:C_1206_3216Metric"
 			(at 186.3852 147.32 0)
 			(effects
@@
 	(symbol
 		(lib_id "JS202011SCQN:JS202011SCQN")
-		(at 146.05 45.72 0)
+		(at 147.32 48.26 0)
 		(unit 1)
 		(exclude_from_sim no)
@@
 		(fields_autoplaced yes)
 		(property "Reference" "S1"
-			(at 156.21 38.1 0)
+			(at 157.48 40.64 0)
 			(effects
 				(font
@@
 		)
 		(property "Value" "JS202011SCQN"
-			(at 156.21 40.64 0)
+			(at 157.48 43.18 0)
 			(effects
 				(font
@@
 		)
 		(property "Footprint" "JS202011SCQN:JS202011SCQN"
-			(at 162.56 140.64 0)
+			(at 163.83 143.18 0)
 			(effects
 				(font
@@
 		)
 		(property "Datasheet" "https://www.ckswitches.com/media/1422/js.pdf"
-			(at 162.56 240.64 0)
+			(at 163.83 243.18 0)
 			(effects
 				(font
@@
 		)
 		(property "Description" "Sub miniature slide switches"
-			(at 146.05 45.72 0)
+			(at 147.32 48.26 0)
 			(effects
 				(font
@@
 		)
 		(property "Height" "5.5"
-			(at 162.56 440.64 0)
+			(at 163.83 443.18 0)
 			(effects
 				(font
@@
 		)
 		(property "Mouser Part Number" "611-JS202011SCQN"
-			(at 162.56 540.64 0)
+			(at 163.83 543.18 0)
 			(effects
 				(font
@@
 		)
 		(property "Mouser Price/Stock" "https://www.mouser.co.uk/ProductDetail/CK/JS202011SCQN?qs=LgMIjt8LuD95JYWxZ7NvZA%3D%3D"
-			(at 162.56 640.64 0)
+			(at 163.83 643.18 0)
 			(effects
 				(font
@@
 		)
 		(property "Manufacturer_Name" "C & K COMPONENTS"
-			(at 162.56 740.64 0)
+			(at 163.83 743.18 0)
 			(effects
 				(font
@@
 		)
 		(property "Manufacturer_Part_Number" "JS202011SCQN"
-			(at 162.56 840.64 0)
+			(at 163.83 843.18 0)
 			(effects
 				(font
@@
 			)
 		)
-		(property "Footprint" "Capacitor_SMD:C_0603_1608Metric"
+		(property "Footprint" "Capacitor_SMD:C_0805_2012Metric"
 			(at 159.7152 147.32 0)
 			(effects
@@
 			)
 		)
-		(property "Footprint" "Resistor_SMD:R_0603_1608Metric"
+		(property "Footprint" "Resistor_SMD:R_1206_3216Metric"
 			(at 174.752 134.62 90)
 			(effects
@@
 			)
 		)
-		(property "Footprint" "Capacitor_SMD:C_0603_1608Metric"
+		(property "Footprint" "Capacitor_SMD:C_0402_1005Metric"
 			(at 31.4452 106.68 0)
 			(effects
@@
 			)
 		)
-		(property "Footprint" "Resistor_SMD:R_0603_1608Metric"
+		(property "Footprint" "Resistor_SMD:R_1206_3216Metric"
 			(at 156.972 134.62 90)
 			(effects
@@
 			)
 		)
-		(property "Footprint" "Capacitor_SMD:C_0603_1608Metric"
+		(property "Footprint" "Capacitor_SMD:C_1210_3225Metric"
 			(at 168.6052 147.32 0)
 			(effects
@@
 	(symbol
 		(lib_id "Device:R")
-		(at 181.61 40.64 0)
+		(at 182.88 43.18 0)
 		(unit 1)
 		(exclude_from_sim no)
@@
 		(dnp no)
 		(property "Reference" "R1"
-			(at 183.134 39.37 0)
+			(at 184.404 41.91 0)
 			(effects
 				(font
@@
 		)
 		(property "Value" "33k"
-			(at 183.134 41.91 0)
+			(at 184.404 44.45 0)
 			(effects
 				(font
@@
 		)
 		(property "Footprint" "Resistor_SMD:R_0603_1608Metric"
-			(at 179.832 40.64 90)
+			(at 181.102 43.18 90)
 			(effects
 				(font
@@
 		)
 		(property "Datasheet" "~"
-			(at 181.61 40.64 0)
+			(at 182.88 43.18 0)
 			(effects
 				(font
@@
 		)
 		(property "Description" "Resistor"
-			(at 181.61 40.64 0)
+			(at 182.88 43.18 0)
 			(effects
 				(font
@@
 			)
 		)
-		(property "Value" "505k"
+		(property "Value" "205k"
 			(at 128.524 135.89 0)
 			(effects
@@
 	(symbol
 		(lib_id "power:GND")
-		(at 181.61 55.88 0)
+		(at 182.88 58.42 0)
 		(unit 1)
 		(exclude_from_sim no)
@@
 		(dnp no)
 		(property "Reference" "#PWR07"
-			(at 181.61 62.23 0)
+			(at 182.88 64.77 0)
 			(effects
 				(font
@@
 		)
 		(property "Value" "GND"
-			(at 181.61 59.69 0)
+			(at 182.88 62.23 0)
 			(effects
 				(font
@@
 		)
 		(property "Footprint" ""
-			(at 181.61 55.88 0)
+			(at 182.88 58.42 0)
 			(effects
 				(font
@@
 		)
 		(property "Datasheet" ""
-			(at 181.61 55.88 0)
+			(at 182.88 58.42 0)
 			(effects
 				(font
@@
 		)
 		(property "Description" "Power symbol creates a global label with name \"GND\" , ground"
-			(at 181.61 55.88 0)
+			(at 182.88 58.42 0)
 			(effects
 				(font
@@
 			)
 		)
-		(property "Footprint" "Capacitor_SMD:C_0603_1608Metric"
+		(property "Footprint" "Capacitor_SMD:C_0402_1005Metric"
 			(at 31.4452 151.13 0)
 			(effects
@@
 			)
 		)
-		(property "Footprint" "Capacitor_SMD:C_0603_1608Metric"
+		(property "Footprint" "Capacitor_SMD:C_1206_3216Metric"
 			(at 177.4952 147.32 0)
 			(effects
@@
 			)
 		)
-		(property "Footprint" "Resistor_SMD:R_0603_1608Metric"
+		(property "Footprint" "Resistor_SMD:R_1206_3216Metric"
 			(at 148.082 134.62 90)
 			(effects
@@
 			)
 		)
-		(property "Footprint" "Resistor_SMD:R_0603_1608Metric"
+		(property "Footprint" "Resistor_SMD:R_1206_3216Metric"
 			(at 165.862 134.62 90)
 			(effects
@@
 			)
 		)
-		(property "Value" "100nF"
+		(property "Value" "22uF"
 			(at 57.658 53.34 0)
 			(effects
@@
 			)
 		)
-		(property "Footprint" "Capacitor_SMD:C_0603_1608Metric"
+		(property "Footprint" "Capacitor_SMD:C_1206_3216Metric"
 			(at 58.1152 54.61 0)
 			(effects
@@
 			)
 		)
-		(property "Footprint" "Capacitor_SMD:C_1206_3216Metric"
+		(property "Footprint" "Capacitor_SMD:C_0805_2012Metric"
 			(at 86.0552 54.61 0)
 			(effects
@@
 			)
 		)
-		(property "Value" "135k"
+		(property "Value" "54.9k"
 			(at 128.524 153.67 0)
 			(effects
