File: kicad_proj/fpga_pre_test.kicad_pcb (KiCad board)
At the start: 2 copper layers, 50.5 x 34.8 mm, 50 parts, among them IC1 ZMR330FTA, IC2 LM3880MFX-1AB_NOPB, IC3 TPS62147RGXT, IC4 TPS62147RGXT, J1 T50201500000G, J2 T50201500000G, Y1 ASDMB-25.000MHZ-XY-T

Commit message: Update PCB design and cost information
Routing:
- net /3V3LVR: track 18.1 -> 24.8 mm
- net /VOUT1: track 12.6 -> 13.9 mm, vias 1 -> 2
Changed lines of the file:
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@@
 	)
 	(setup
+		(stackup
+			(layer "F.SilkS"
+				(type "Top Silk Screen")
+			)
+			(layer "F.Paste"
+				(type "Top Solder Paste")
+			)
+			(layer "F.Mask"
+				(type "Top Solder Mask")
+				(thickness 0.01)
+			)
+			(layer "F.Cu"
+				(type "copper")
+				(thickness 0.035)
+			)
+			(layer "dielectric 1"
+				(type "core")
+				(thickness 1.51)
+				(material "FR4")
+				(epsilon_r 4.5)
+				(loss_tangent 0.02)
+			)
+			(layer "B.Cu"
+				(type "copper")
+				(thickness 0.035)
+			)
+			(layer "B.Mask"
+				(type "Bottom Solder Mask")
+				(thickness 0.01)
+			)
+			(layer "B.Paste"
+				(type "Bottom Solder Paste")
+			)
+			(layer "B.SilkS"
+				(type "Bottom Silk Screen")
+			)
+			(copper_finish "None")
+			(dielectric_constraints no)
+		)
 		(pad_to_mask_clearance 0)
 		(allow_soldermask_bridges_in_footprints no)
@@
 			(at 1.65 0 0)
 			(layer "F.SilkS")
+			(hide yes)
 			(effects
 				(font
@@
 			(layer "F.Fab")
 		)
-		(fp_text user "${REFERENCE}"
-			(at 1.65 0 0)
-			(layer "F.Fab")
-			(effects
-				(font
-					(size 1.27 1.27)
-					(thickness 0.254)
-				)
-			)
-		)
 		(pad "1" thru_hole circle
 			(at 0 0 180)
@@
 			(at 0 0 90)
 			(layer "F.SilkS")
+			(hide yes)
 			(effects
 				(font
@@
 			(layer "F.Fab")
 		)
-		(fp_text user "${REFERENCE}"
-			(at 0 0 90)
-			(layer "F.Fab")
-			(effects
-				(font
-					(size 1.27 1.27)
-					(thickness 0.254)
-				)
-			)
-		)
 		(pad "1" smd rect
 			(at -1 0 270)
@@
 	)
 	(segment
+		(start 141.36 99.96)
+		(end 139.32 99.96)
+		(width 0.5)
+		(layer "B.Cu")
+		(net 3)
+	)
+	(segment
 		(start 136.340114 101.682499)
 		(end 136.848735 101.682499)
@@
 	)
 	(segment
+		(start 141.931493 100.531493)
+		(end 141.36 99.96)
+		(width 0.5)
+		(layer "B.Cu")
+		(net 3)
+	)
+	(segment
 		(start 141.931493 101.162499)
 		(end 141.931493 104.082499)
@@
 	)
 	(segment
+		(start 141.931493 101.162499)
+		(end 141.931493 100.531493)
+		(width 0.5)
+		(layer "B.Cu")
+		(net 3)
+	)
+	(segment
+		(start 137.597501 101.682499)
+		(end 136.848735 101.682499)
+		(width 0.5)
+		(layer "B.Cu")
+		(net 3)
+	)
+	(segment
+		(start 139.32 99.96)
+		(end 137.597501 101.682499)
+		(width 0.5)
+		(layer "B.Cu")
+		(net 3)
+	)
+	(segment
 		(start 130.52 96.13)
 		(end 131.77 96.13)
@@
 	)
 	(via
+		(at 144.915 88.14)
+		(size 0.5)
+		(drill 0.3)
+		(layers "F.Cu" "B.Cu")
+		(net 5)
+	)
+	(via
 		(at 141.175 88.49)
 		(size 0.45)
@@
 		(net 5)
 	)
+	(segment
+		(start 144.915 88.14)
+		(end 144.915 86.92)
+		(width 0.5)
+		(layer "B.Cu")
+		(net 5)
+	)
